Commit message: updated robot_core.xacro

File: description/robot_core.xacro (robot description, xacro)
@@ -2,4 +2,30 @@
 <robot xmlns:xacro="http://www.ros.org/wiki/xacro"  name="robot">
     <material name="white" >
-    <
+        <color rgba="1 1 1 1"/>
+    </material>
+    <material name="orange" >
+        <color rgba="1 0.3 0.1 1"/>
+    </material>
+    <material name="blue" >
+        <color rgba="0.2 0.2 1 1"/>
+    </material>
+    <material name="black" >
+        <color rgba="0 0 0 1"/>
+    </material>
+    <link name="base_link">
+    </link>
+    <joint name="chassis_joint" type="fixed">
+        <parent link="base_link"/>
+        <child link="chassis"/>
+        <origin xyz="-0.1 0 0"/>
+    </joint>
+    <link name="chassis">
+        <visual>
+            <origin xyz="0.15 0 0.075"/>
+            <geometry>
+                <box size="0.3 0.3 0.15"/>
+            </geometry>
+            <material name="white"/>
+        </visual>
+    </link>
 </robot>

Commit message: updated pat_bot

File: description/robot_core.xacro (robot description, xacro)
@@ -13,6 +13,8 @@
         <color rgba="0 0 0 1"/>
     </material>
+    <!-- BASE  LINK -->
     <link name="base_link">
     </link>
+    <!-- CHASSIS LINK -->
     <joint name="chassis_joint" type="fixed">
         <parent link="base_link"/>
@@ -29,3 +31,47 @@
         </visual>
     </link>
+    <!-- LEFT WHEEL LINK -->
+    <joint name="left_wheel_joint" type="continuous">
+        <parent link="base_link"/>
+        <child link="left_wheel"/>
+        <origin xyz="0 0.175 0" rpy="-${pi/2} 0 0"/>
+        <axis xyz="0 0 1"/>
+    </joint>
+    <link name="left_wheel">
+        <visual>
+            <geometry>
+                <cyclinder radius="0.05" length="0.04"/>
+            </geometry>
+            <material name="blue"/>
+        </visual>
+    </link>
+    <!-- RIGHT WHEEL LINK -->
+    <joint name="right_wheel_joint" type="continuous">
+        <parent link="base_link"/>
+        <child link="right_wheel"/>
+        <origin xyz="0 -0.175 0" rpy="${pi/2} 0 0"/>
+        <axis xyz="0 0 -1"/>
+    </joint>
+    <link name="right_wheel">
+        <visual>
+            <geometry>
+                <cyclinder radius="0.05" length="0.04"/>
+            </geometry>
+            <material name="blue"/>
+        </visual>
+    </link>
+    <!-- CASTER WHEEL LINK -->
+    <joint name="caster_wheel_joint" type="fixed">
+        <parent link="chassis"/>
+        <child link="caster_wheel"/>
+        <origin xyz="0.24 0 0"/>
+    </joint>
+    <link name="caster_wheel">
+        <visual>
+            <geometry>
+                <sphere radius="0.05"/>
+            </geometry>
+            <material name="black"/>
+        </visual>
+    </link>
 </robot>

Commit message: updated pat_bot

File: description/robot_core.xacro (robot description, xacro)
@@ -41,5 +41,5 @@
         <visual>
             <geometry>
-                <cyclinder radius="0.05" length="0.04"/>
+                <cylinder radius="0.05" length="0.04"/>
             </geometry>
             <material name="blue"/>
@@ -56,5 +56,5 @@
         <visual>
             <geometry>
-                <cyclinder radius="0.05" length="0.04"/>
+                <cylinder radius="0.05" length="0.04"/>
             </geometry>
             <material name="blue"/>

Commit message: included inertial macros

File: description/robot_core.xacro (robot description, xacro)
@@ -1,4 +1,5 @@
 <?xml version="1.0"?>
 <robot xmlns:xacro="http://www.ros.org/wiki/xacro"  name="robot">
+    <xacro:include filename="inertial_macro.xarco"/>
     <material name="white" >
         <color rgba="1 1 1 1"/>
@@ -36,4 +37,7 @@
             </geometry>
         </collision>
+        <xacro:inertial_box mass="0.5" x="0.3" y="0.3" z="0.15">
+            <origin xyz="0.15 0 0.075" rpy="0 0 0"/>
+        </xacro:inertial_box>
     </link>
     <!-- LEFT WHEEL LINK -->
@@ -56,4 +60,7 @@
             </geometry>
         </collision>
+        <xacro:inertial_cylinder mass="0.1" length="0.04" radius="0.05">
+            <origin xyz="0 0 0" rpy="0 0 0"/>
+        </xacro:inertial_cylinder>
     </link>
     <!-- RIGHT WHEEL LINK -->
@@ -76,4 +83,7 @@
             </geometry>
         </collision>
+        <xacro:inertial_cylinder mass="0.1" length="0.04" radius="0.05">
+            <origin xyz="0 0 0" rpy="0 0 0"/>
+        </xacro:inertial_cylinder>
     </link>
     <!-- CASTER WHEEL LINK -->
@@ -95,4 +105,7 @@
             </geometry>
         </collision>
+        <xacro:inertial_sphere mass="0.1" radius="0.05">
+            <origin xyz="0 0 0" rpy="0 0 0"/>
+        </xacro:inertial_sphere>
     </link>
 </robot>
