Commit message: update

File: description/robot.urdf.xacro (robot description, xacro)
@@ -1,6 +1,4 @@
 <?xml version="1.0"?>
 <robot xmlns:xacro="http://www.ros.org/wiki/xacro"  name="robot">
-    <!-- Example link -->
-    <link name="base_link"></link>
     <xacro:include filename="robot_core.xacro" />
 </robot>

Commit message: included camera, depth camera, lidar

File: description/robot.urdf.xacro (robot description, xacro)
@@ -2,4 +2,8 @@
 <robot xmlns:xacro="http://www.ros.org/wiki/xacro"  name="robot">
     <xacro:include filename="robot_core.xacro" />
-    <xacro:include filename="gazebo_control.xacro"/>
+    <!-- <xacro:include filename="gazebo_control.xacro"/> -->
+    <xacro:include filename="ros2_control.xacro"/>
+    <xacro:include filename="lidar.xacro"/>
+    <!-- <xacro:include filename="camera.xacro"/> -->
+    <xacro:include filename="depth_camera.xacro"/>
 </robot>

File: description/robot_core.xacro (robot description, xacro)
@@ -13,4 +13,7 @@
     <material name="black" >
         <color rgba="0 0 0 1"/>
+    </material>
+    <material name="red" >
+        <color rgba="1 0 0 1"/>
     </material>
     <!-- BASE  LINK -->

Commit message: introduced: beginning of joystick control, nav2, and slamtoolbox

File: description/robot.urdf.xacro (robot description, xacro)
@@ -1,7 +1,12 @@
 <?xml version="1.0"?>
 <robot xmlns:xacro="http://www.ros.org/wiki/xacro"  name="robot">
-    <xacro:include filename="robot_core.xacro" />
-    <!-- <xacro:include filename="gazebo_control.xacro"/> -->
-    <xacro:include filename="ros2_control.xacro"/>
+    <xacro:include filename="robot_core.xacro"/>
+    <xacro:arg name="use_ros2_control" default="true"/>
+    <xacro:if value="$(arg use_ros2_control)">
+        <xacro:include filename="ros2_control.xacro"/>
+    </xacro:if>
+    <xacro:unless value="$(arg use_ros2_control)">
+        <xacro:include filename="gazebo_control.xacro"/>
+    </xacro:unless>
     <xacro:include filename="lidar.xacro"/>
     <!-- <xacro:include filename="camera.xacro"/> -->

File: description/robot_core.xacro (robot description, xacro)
@@ -18,5 +18,12 @@
     </material>
     <!-- BASE  LINK -->
-    <link name="base_link">
+    <link name="base_link"></link>
+    <!-- BASE_FOOTPRINT LINK -->
+    <joint name="base_footprint_joint" type="fixed">
+        <parent link="base_link"/>
+        <child link="base_footprint"/>
+        <origin xyz="0 0 0" rpy="0 0 0"/>
+    </joint>
+    <link name="base_footprint">
     </link>
     <!-- CHASSIS LINK -->
@@ -63,5 +70,6 @@
         <collision>
             <geometry>
-                <cylinder radius="0.05" length="0.04"/>
+                <!-- <cylinder radius="0.05" length="0.04"/> -->
+                <sphere radius="0.05"/>
             </geometry>
         </collision>
@@ -89,5 +97,6 @@
         <collision>
             <geometry>
-                <cylinder radius="0.05" length="0.04"/>
+                <!-- <cylinder radius="0.05" length="0.04"/> -->
+                <sphere radius="0.05"/>
             </geometry>
         </collision>

File: description/ros2_control.xacro (robot description, xacro)
@@ -3,4 +3,5 @@
     <ros2_control name="GazeboSystem" type="system">
         <hardware>
+            <!-- this is the hardware interface -->
             <plugin>gazebo_ros2_control/GazeboSystem</plugin>
         </hardware>
@@ -22,3 +23,8 @@
         </joint>
     </ros2_control>
+    <gazebo>
+        <plugin name="gazebo_ros2_control" filename="libgazebo_ros2_control.so">
+            <parameters>$(find pat_bot)/config/my_controllers.yaml</parameters>
+        </plugin>
+    </gazebo>
 </robot>
